File: chainclock.sch (EAGLE design)
At the start: 14 parts

Commit message: Move around voltage reg
Parts:
- added C5, C6: .01uf, SparkFun-Capacitors:CAPKIT
- added R11, R12, R5, R6: 10k, SparkFun-Resistors:RESISTOR2010
- added SW1: ROTARTY_ENCODER, SparkFun-Electromechanical:ROTARTY_ENCODER
- renumbered U$1 to PTN0405
Connections:
- removed net VIN: C3.+, PTN0405.VIN
- new net N$2: R11.1, R5.1, SW1.B
- new net N$5: R12.1, R6.2, SW1.A
- new net RENBTN: ARDUNOFIO.D6, SW1.SW+
- new net RENCA: ARDUNOFIO.D12, C5.1, R6.1
- new net RENCB: ARDUNOFIO.D11, C6.1, R5.2
- net 3V31: now also C3.+, PTN0405.VIN
- net 3V32: now also R11.2, R12.2
- net GND: now also C5.2, C6.2, SW1.C, SW1.SW-
Changed lines of the file:
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@@
 <part name="R3" library="SparkFun-Resistors" deviceset="RESISTOR" device="EZ" value="10k"/>
 <part name="GND5" library="SparkFun-Aesthetics" deviceset="GND" device=""/>
-<part name="U$1" library="desjardins" deviceset="PTN0405C" device=""/>
+<part name="PTN0405" library="desjardins" deviceset="PTN0405C" device=""/>
 <part name="C3" library="SparkFun-Passives" deviceset="CAP_POL" device="PTH1"/>
 <part name="C4" library="SparkFun-Passives" deviceset="CAP_POL" device="PTH1"/>
@@
 <part name="GND8" library="SparkFun-Aesthetics" deviceset="GND" device=""/>
 <part name="FRAME1" library="frames" deviceset="FRAME_A_L" device=""/>
+<part name="SW1" library="SparkFun-Electromechanical" deviceset="ROTARTY_ENCODER" device=""/>
+<part name="GND7" library="SparkFun-Aesthetics" deviceset="GND" device=""/>
+<part name="C5" library="SparkFun-Capacitors" deviceset="CAP" device="KIT" value=".01uf"/>
+<part name="C6" library="SparkFun-Capacitors" deviceset="CAP" device="KIT" value=".01uf"/>
+<part name="GND10" library="SparkFun-Aesthetics" deviceset="GND" device=""/>
+<part name="GND11" library="SparkFun-Aesthetics" deviceset="GND" device=""/>
+<part name="R11" library="SparkFun-Resistors" deviceset="RESISTOR" device="2010" value="10k"/>
+<part name="R12" library="SparkFun-Resistors" deviceset="RESISTOR" device="2010" value="10k"/>
+<part name="GND12" library="SparkFun-Aesthetics" deviceset="GND" device=""/>
+<part name="R5" library="SparkFun-Resistors" deviceset="RESISTOR" device="2010" value="10k"/>
+<part name="R6" library="SparkFun-Resistors" deviceset="RESISTOR" device="2010" value="10k"/>
 </parts>
 <sheets>
@@
 <instance part="R3" gate="G$1" x="190.5" y="185.42" rot="R270"/>
 <instance part="GND5" gate="1" x="190.5" y="175.26"/>
-<instance part="U$1" gate="G$1" x="45.72" y="137.16"/>
+<instance part="PTN0405" gate="G$1" x="45.72" y="137.16"/>
 <instance part="C3" gate="G$1" x="20.32" y="134.62" rot="R270"/>
 <instance part="C4" gate="G$1" x="71.12" y="142.24" rot="R90"/>
@@
 <instance part="FRAME1" gate="G$1" x="0" y="0"/>
 <instance part="FRAME1" gate="G$2" x="172.72" y="0"/>
+<instance part="SW1" gate="G$1" x="71.12" y="83.82" rot="MR90"/>
+<instance part="GND7" gate="1" x="71.12" y="99.06" rot="R180"/>
+<instance part="C5" gate="G$1" x="50.8" y="88.9" rot="MR0"/>
+<instance part="C6" gate="G$1" x="91.44" y="88.9" rot="MR0"/>
+<instance part="GND10" gate="1" x="91.44" y="81.28" rot="MR0"/>
+<instance part="GND11" gate="1" x="50.8" y="81.28" rot="MR0"/>
+<instance part="R11" gate="G$1" x="76.2" y="106.68" rot="MR90"/>
+<instance part="R12" gate="G$1" x="66.04" y="106.68" rot="MR90"/>
+<instance part="GND12" gate="1" x="66.04" y="68.58"/>
+<instance part="R5" gate="G$1" x="83.82" y="96.52" rot="MR180"/>
+<instance part="R6" gate="G$1" x="58.42" y="96.52" rot="MR180"/>
 </instances>
 <busses>
@@
 </segment>
 <segment>
-<pinref part="U$1" gate="G$1" pin="GND"/>
+<pinref part="PTN0405" gate="G$1" pin="GND"/>
 <wire x1="27.94" y1="142.24" x2="12.7" y2="142.24" width="0.1524" layer="91"/>
 <wire x1="12.7" y1="142.24" x2="12.7" y2="134.62" width="0.1524" layer="91"/>
@@
 <wire x1="78.74" y1="142.24" x2="78.74" y2="132.08" width="0.1524" layer="91"/>
 <junction x="78.74" y="132.08"/>
+</segment>
+<segment>
+<pinref part="SW1" gate="G$1" pin="C"/>
+<wire x1="71.12" y1="93.98" x2="71.12" y2="96.52" width="0.1524" layer="91"/>
+<pinref part="GND7" gate="1" pin="GND"/>
+</segment>
+<segment>
+<pinref part="C6" gate="G$1" pin="2"/>
+<wire x1="91.44" y1="86.36" x2="91.44" y2="83.82" width="0.1524" layer="91"/>
+<pinref part="GND10" gate="1" pin="GND"/>
+</segment>
+<segment>
+<pinref part="C5" gate="G$1" pin="2"/>
+<wire x1="50.8" y1="86.36" x2="50.8" y2="83.82" width="0.1524" layer="91"/>
+<pinref part="GND11" gate="1" pin="GND"/>
+</segment>
+<segment>
+<pinref part="SW1" gate="G$1" pin="SW-"/>
+<wire x1="66.04" y1="73.66" x2="66.04" y2="71.12" width="0.1524" layer="91"/>
+<pinref part="GND12" gate="1" pin="GND"/>
 </segment>
 </net>
@@
 <pinref part="ARDUNOFIO" gate="G$1" pin="D10"/>
 <wire x1="43.18" y1="193.04" x2="45.72" y2="193.04" width="0.1524" layer="91"/>
+<label x="43.18" y="193.04" size="1.778" layer="95"/>
 </segment>
 </net>
@@
 <label x="7.62" y="172.72" size="1.778" layer="95"/>
 </segment>
+<segment>
+<pinref part="PTN0405" gate="G$1" pin="VIN"/>
+<label x="27.94" y="124.46" size="1.778" layer="95" rot="MR0"/>
+<pinref part="C3" gate="G$1" pin="+"/>
+<wire x1="27.94" y1="134.62" x2="25.4" y2="134.62" width="0.1524" layer="91"/>
+<wire x1="25.4" y1="134.62" x2="22.86" y2="134.62" width="0.1524" layer="91"/>
+<wire x1="25.4" y1="134.62" x2="25.4" y2="127" width="0.1524" layer="91"/>
+<junction x="25.4" y="134.62"/>
+</segment>
 </net>
 <net name="3V32" class="0">
@@
 <label x="170.18" y="200.66" size="1.778" layer="95"/>
 </segment>
-</net>
-<net name="VIN" class="0">
-<segment>
-<pinref part="U$1" gate="G$1" pin="VIN"/>
-<label x="22.86" y="134.62" size="1.778" layer="95"/>
-<pinref part="C3" gate="G$1" pin="+"/>
-<wire x1="27.94" y1="134.62" x2="22.86" y2="134.62" width="0.1524" layer="91"/>
+<segment>
+<wire x1="76.2" y1="111.76" x2="76.2" y2="114.3" width="0.1524" layer="91"/>
+<wire x1="76.2" y1="114.3" x2="71.12" y2="114.3" width="0.1524" layer="91"/>
+<wire x1="71.12" y1="114.3" x2="66.04" y2="114.3" width="0.1524" layer="91"/>
+<wire x1="66.04" y1="114.3" x2="66.04" y2="111.76" width="0.1524" layer="91"/>
+<wire x1="71.12" y1="114.3" x2="71.12" y2="116.84" width="0.1524" layer="91"/>
+<junction x="71.12" y="114.3"/>
+<label x="48.26" y="127" size="1.778" layer="95"/>
+<pinref part="R11" gate="G$1" pin="2"/>
+<pinref part="R12" gate="G$1" pin="2"/>
 </segment>
 </net>
 <net name="VDD12" class="0">
 <segment>
-<pinref part="U$1" gate="G$1" pin="VOUT"/>
+<pinref part="PTN0405" gate="G$1" pin="VOUT"/>
 <wire x1="63.5" y1="142.24" x2="66.04" y2="142.24" width="0.1524" layer="91"/>
 <pinref part="C4" gate="G$1" pin="+"/>
@@
 <net name="N$3" class="0">
 <segment>
-<pinref part="U$1" gate="G$1" pin="VOADJ"/>
+<pinref part="PTN0405" gate="G$1" pin="VOADJ"/>
 <wire x1="63.5" y1="132.08" x2="66.04" y2="132.08" width="0.1524" layer="91"/>
 <pinref part="R4" gate="G$1" pin="1"/>
 </segment>
 </net>
+<net name="N$2" class="0">
+<segment>
+<pinref part="SW1" gate="G$1" pin="B"/>
+<wire x1="76.2" y1="93.98" x2="76.2" y2="96.52" width="0.1524" layer="91"/>
+<wire x1="76.2" y1="96.52" x2="78.74" y2="96.52" width="0.1524" layer="91"/>
+<wire x1="76.2" y1="96.52" x2="76.2" y2="101.6" width="0.1524" layer="91"/>
+<junction x="76.2" y="96.52"/>
+<pinref part="R11" gate="G$1" pin="1"/>
+<pinref part="R5" gate="G$1" pin="1"/>
+</segment>
+</net>
+<net name="N$5" class="0">
+<segment>
+<pinref part="SW1" gate="G$1" pin="A"/>
+<wire x1="66.04" y1="93.98" x2="66.04" y2="96.52" width="0.1524" layer="91"/>
+<wire x1="66.04" y1="96.52" x2="63.5" y2="96.52" width="0.1524" layer="91"/>
+<wire x1="66.04" y1="96.52" x2="66.04" y2="101.6" width="0.1524" layer="91"/>
+<junction x="66.04" y="96.52"/>
+<pinref part="R12" gate="G$1" pin="1"/>
+<pinref part="R6" gate="G$1" pin="2"/>
+</segment>
+</net>
+<net name="RENBTN" class="0">
+<segment>
+<pinref part="ARDUNOFIO" gate="G$1" pin="D6"/>
+<wire x1="43.18" y1="182.88" x2="45.72" y2="182.88" width="0.1524" layer="91"/>
+<label x="43.18" y="182.88" size="1.778" layer="95"/>
+</segment>
+<segment>
+<pinref part="SW1" gate="G$1" pin="SW+"/>
+<wire x1="76.2" y1="73.66" x2="76.2" y2="71.12" width="0.1524" layer="91"/>
+<label x="73.66" y="68.58" size="1.778" layer="95"/>
+</segment>
+</net>
+<net name="RENCB" class="0">
+<segment>
+<pinref part="ARDUNOFIO" gate="G$1" pin="D11"/>
+<wire x1="43.18" y1="195.58" x2="45.72" y2="195.58" width="0.1524" layer="91"/>
+<label x="43.18" y="195.58" size="1.778" layer="95"/>
+</segment>
+<segment>
+<wire x1="88.9" y1="96.52" x2="91.44" y2="96.52" width="0.1524" layer="91"/>
+<wire x1="91.44" y1="96.52" x2="93.98" y2="96.52" width="0.1524" layer="91"/>
+<wire x1="91.44" y1="96.52" x2="91.44" y2="93.98" width="0.1524" layer="91"/>
+<junction x="91.44" y="96.52"/>
+<pinref part="C6" gate="G$1" pin="1"/>
+<label x="101.6" y="96.52" size="1.778" layer="95" rot="MR0"/>
+<pinref part="R5" gate="G$1" pin="2"/>
+</segment>
+</net>
+<net name="RENCA" class="0">
+<segment>
+<pinref part="ARDUNOFIO" gate="G$1" pin="D12"/>
+<wire x1="43.18" y1="198.12" x2="45.72" y2="198.12" width="0.1524" layer="91"/>
+<label x="43.18" y="198.12" size="1.778" layer="95"/>
+</segment>
+<segment>
+<wire x1="53.34" y1="96.52" x2="50.8" y2="96.52" width="0.1524" layer="91"/>
+<wire x1="50.8" y1="96.52" x2="48.26" y2="96.52" width="0.1524" layer="91"/>
+<wire x1="50.8" y1="96.52" x2="50.8" y2="93.98" width="0.1524" layer="91"/>
+<junction x="50.8" y="96.52"/>
+<pinref part="C5" gate="G$1" pin="1"/>
+<label x="48.26" y="96.52" size="1.778" layer="95" rot="MR0"/>
+<pinref part="R6" gate="G$1" pin="1"/>
+</segment>
+</net>

Commit message: Switch out crystal
Parts:
- removed C1, C2: 33pf, SparkFun-Capacitors:0.1UF-50V-20%(PTH)KIT-EZ
- removed Q1: (no value), adafruit:CRYSTALTC26H
- removed R1: 330, SparkFun-Resistors:RESISTOREZ
- removed R2: 10M, SparkFun-Resistors:RESISTOREZ
- added U$4: SG30XXJC, desjardins:SG30XXJC
Connections:
- removed net N$1: C2.1, Q1.1, R1.1
- removed net RS: C1.1, COUNTER.RS, Q1.2, R2.2
- net 3V32: now also U$4.VCC, U$4.VIO
- net GND: now also U$4.GND; no longer C1.2, C2.2
- net RTC: now also U$4.OUT; no longer R1.2, R2.1
Other:
- moved on the sheet: COUNTER
Changed lines of the file:
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@@
 <part name="COUNTER" library="desjardins" deviceset="4060" device=""/>
 <part name="ARDUNOFIO" library="desjardins" deviceset="ARDUINOFIO" device=""/>
-<part name="R1" library="SparkFun-Resistors" deviceset="RESISTOR" device="EZ" value="330"/>
-<part name="R2" library="SparkFun-Resistors" deviceset="RESISTOR" device="EZ" value="10M"/>
-<part name="C1" library="SparkFun-Capacitors" deviceset="0.1UF-50V-20%(PTH)" device="KIT-EZ" value="33pf"/>
-<part name="C2" library="SparkFun-Capacitors" deviceset="0.1UF-50V-20%(PTH)" device="KIT-EZ" value="33pf"/>
-<part name="Q1" library="adafruit" deviceset="CRYSTAL" device="TC26H"/>
-<part name="GND1" library="SparkFun-Aesthetics" deviceset="GND" device=""/>
 <part name="HBRIDGE" library="desjardins" deviceset="SN754410" device=""/>
 <part name="GND2" library="SparkFun-Aesthetics" deviceset="GND" device=""/>
@@
 <part name="R5" library="SparkFun-Resistors" deviceset="RESISTOR" device="2010" value="10k"/>
 <part name="R6" library="SparkFun-Resistors" deviceset="RESISTOR" device="2010" value="10k"/>
+<part name="GND1" library="SparkFun-Aesthetics" deviceset="GND" device=""/>
+<part name="U$4" library="desjardins" deviceset="SG30XX" device="JC"/>
 </parts>
 <sheets>
@@
 </plain>
 <instances>
-<instance part="COUNTER" gate="G$1" x="101.6" y="180.34"/>
+<instance part="COUNTER" gate="G$1" x="68.58" y="182.88"/>
 <instance part="ARDUNOFIO" gate="G$1" x="27.94" y="182.88" rot="R90"/>
-<instance part="R1" gate="G$1" x="60.96" y="190.5" rot="R90"/>
-<instance part="R2" gate="G$1" x="68.58" y="198.12"/>
-<instance part="C1" gate="G$1" x="76.2" y="175.26"/>
-<instance part="C2" gate="G$1" x="60.96" y="175.26"/>
-<instance part="Q1" gate="G$1" x="68.58" y="182.88"/>
-<instance part="GND1" gate="1" x="68.58" y="165.1"/>
 <instance part="HBRIDGE" gate="G$1" x="154.94" y="177.8"/>
-<instance part="GND2" gate="1" x="121.92" y="182.88" rot="R90"/>
+<instance part="GND2" gate="1" x="88.9" y="185.42" rot="R90"/>
 <instance part="GND3" gate="1" x="132.08" y="180.34" rot="R270"/>
 <instance part="GND4" gate="1" x="177.8" y="180.34" rot="R90"/>
@@
 <instance part="R5" gate="G$1" x="83.82" y="96.52" rot="MR180"/>
 <instance part="R6" gate="G$1" x="58.42" y="96.52" rot="MR180"/>
+<instance part="GND1" gate="1" x="88.9" y="149.86" rot="R270"/>
+<instance part="U$4" gate="G$1" x="106.68" y="154.94"/>
 </instances>
 <busses>
@@
 <net name="GND" class="0">
 <segment>
-<pinref part="C2" gate="G$1" pin="2"/>
-<wire x1="60.96" y1="172.72" x2="60.96" y2="170.18" width="0.1524" layer="91"/>
-<pinref part="C1" gate="G$1" pin="2"/>
-<wire x1="76.2" y1="172.72" x2="76.2" y2="170.18" width="0.1524" layer="91"/>
-<wire x1="60.96" y1="170.18" x2="68.58" y2="170.18" width="0.1524" layer="91"/>
-<wire x1="76.2" y1="170.18" x2="68.58" y2="170.18" width="0.1524" layer="91"/>
-<wire x1="68.58" y1="170.18" x2="68.58" y2="167.64" width="0.1524" layer="91"/>
-<junction x="68.58" y="170.18"/>
-<pinref part="GND1" gate="1" pin="GND"/>
-</segment>
-<segment>
 <pinref part="COUNTER" gate="G$1" pin="GND"/>
-<wire x1="114.3" y1="187.96" x2="116.84" y2="187.96" width="0.1524" layer="91"/>
+<wire x1="81.28" y1="190.5" x2="83.82" y2="190.5" width="0.1524" layer="91"/>
 <pinref part="COUNTER" gate="G$1" pin="MR"/>
-<wire x1="114.3" y1="182.88" x2="116.84" y2="182.88" width="0.1524" layer="91"/>
-<wire x1="116.84" y1="187.96" x2="116.84" y2="182.88" width="0.1524" layer="91"/>
-<wire x1="116.84" y1="182.88" x2="119.38" y2="182.88" width="0.1524" layer="91"/>
+<wire x1="81.28" y1="185.42" x2="83.82" y2="185.42" width="0.1524" layer="91"/>
+<wire x1="83.82" y1="190.5" x2="83.82" y2="185.42" width="0.1524" layer="91"/>
+<wire x1="83.82" y1="185.42" x2="86.36" y2="185.42" width="0.1524" layer="91"/>
 <pinref part="GND2" gate="1" pin="GND"/>
 </segment>
@@
 <pinref part="GND12" gate="1" pin="GND"/>
 </segment>
-</net>
-<net name="N$1" class="0">
-<segment>
-<pinref part="Q1" gate="G$1" pin="1"/>
-<wire x1="66.04" y1="182.88" x2="60.96" y2="182.88" width="0.1524" layer="91"/>
-<pinref part="C2" gate="G$1" pin="1"/>
-<wire x1="60.96" y1="182.88" x2="60.96" y2="180.34" width="0.1524" layer="91"/>
-<wire x1="60.96" y1="182.88" x2="60.96" y2="185.42" width="0.1524" layer="91"/>
-<pinref part="R1" gate="G$1" pin="1"/>
-<junction x="60.96" y="182.88"/>
-</segment>
-</net>
-<net name="RS" class="0">
-<segment>
-<pinref part="Q1" gate="G$1" pin="2"/>
-<wire x1="71.12" y1="182.88" x2="76.2" y2="182.88" width="0.1524" layer="91"/>
-<pinref part="C1" gate="G$1" pin="1"/>
-<wire x1="76.2" y1="182.88" x2="76.2" y2="180.34" width="0.1524" layer="91"/>
-<wire x1="76.2" y1="182.88" x2="76.2" y2="198.12" width="0.1524" layer="91"/>
-<pinref part="R2" gate="G$1" pin="2"/>
-<wire x1="76.2" y1="198.12" x2="73.66" y2="198.12" width="0.1524" layer="91"/>
-<junction x="76.2" y="182.88"/>
-<wire x1="76.2" y1="198.12" x2="76.2" y2="200.66" width="0.1524" layer="91"/>
-<label x="78.74" y="198.12" size="1.778" layer="95" rot="R90"/>
-</segment>
-<segment>
-<pinref part="COUNTER" gate="G$1" pin="RS"/>
-<wire x1="114.3" y1="177.8" x2="116.84" y2="177.8" width="0.1524" layer="91"/>
-</segment>
-</net>
-<net name="RTC" class="0">
-<segment>
-<pinref part="R1" gate="G$1" pin="2"/>
-<wire x1="60.96" y1="195.58" x2="60.96" y2="198.12" width="0.1524" layer="91"/>
-<wire x1="60.96" y1="198.12" x2="63.5" y2="198.12" width="0.1524" layer="91"/>
-<pinref part="R2" gate="G$1" pin="1"/>
-<wire x1="60.96" y1="198.12" x2="60.96" y2="200.66" width="0.1524" layer="91"/>
-<label x="60.96" y="198.12" size="1.778" layer="95" rot="R90"/>
-</segment>
-<segment>
-<pinref part="COUNTER" gate="G$1" pin="RTC"/>
-<wire x1="114.3" y1="172.72" x2="116.84" y2="172.72" width="0.1524" layer="91"/>
+<segment>
+<wire x1="93.98" y1="149.86" x2="91.44" y2="149.86" width="0.1524" layer="91"/>
+<pinref part="GND1" gate="1" pin="GND"/>
+<pinref part="U$4" gate="G$1" pin="GND"/>
 </segment>
 </net>
@@
 <segment>
 <pinref part="COUNTER" gate="G$1" pin="Q14"/>
-<wire x1="88.9" y1="157.48" x2="86.36" y2="157.48" width="0.1524" layer="91"/>
+<wire x1="55.88" y1="160.02" x2="53.34" y2="160.02" width="0.1524" layer="91"/>
 </segment>
 <segment>
@@
 <segment>
 <pinref part="COUNTER" gate="G$1" pin="VCC"/>
-<wire x1="114.3" y1="193.04" x2="116.84" y2="193.04" width="0.1524" layer="91"/>
-<label x="116.84" y="193.04" size="1.778" layer="95"/>
+<wire x1="81.28" y1="195.58" x2="83.82" y2="195.58" width="0.1524" layer="91"/>
+<label x="83.82" y="195.58" size="1.778" layer="95"/>
 </segment>
 <segment>
@@
 <pinref part="R12" gate="G$1" pin="2"/>
 </segment>
+<segment>
+<wire x1="119.38" y1="160.02" x2="121.92" y2="160.02" width="0.1524" layer="91"/>
+<label x="121.92" y="160.02" size="1.778" layer="95"/>
+<pinref part="U$4" gate="G$1" pin="VCC"/>
+</segment>
+<segment>
+<wire x1="93.98" y1="160.02" x2="91.44" y2="160.02" width="0.1524" layer="91"/>
+<label x="88.9" y="160.02" size="1.778" layer="95"/>
+<pinref part="U$4" gate="G$1" pin="VIO"/>
+</segment>
 </net>
 <net name="VDD12" class="0">
@@
 </segment>
 </net>
+<net name="RTC" class="0">
+<segment>
+<pinref part="COUNTER" gate="G$1" pin="RTC"/>
+<wire x1="81.28" y1="175.26" x2="83.82" y2="175.26" width="0.1524" layer="91"/>
+<label x="81.28" y="175.26" size="1.778" layer="95"/>
+</segment>
+<segment>
+<wire x1="119.38" y1="149.86" x2="121.92" y2="149.86" width="0.1524" layer="91"/>
+<label x="121.92" y="149.86" size="1.778" layer="95"/>
+<pinref part="U$4" gate="G$1" pin="OUT"/>
+</segment>
+</net>

Commit message: Small updates
Other:
- note added: "v1.0"
- moved on the sheet: COUNTER
Changed lines of the file:
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@@
 <text x="175.895" y="25.4" size="2.794" layer="94">Chris Desjardins - cjd@chrisd.info
 http://blog.chrisd.info</text>
+<text x="262.255" y="7.62" size="2.794" layer="94">v1.0</text>
 </plain>
 <instances>
-<instance part="COUNTER" gate="G$1" x="68.58" y="182.88"/>
+<instance part="COUNTER" gate="G$1" x="68.58" y="180.34"/>
 <instance part="ARDUNOFIO" gate="G$1" x="27.94" y="182.88" rot="R90"/>
 <instance part="HBRIDGE" gate="G$1" x="154.94" y="177.8"/>
-<instance part="GND2" gate="1" x="88.9" y="185.42" rot="R90"/>
+<instance part="GND2" gate="1" x="88.9" y="182.88" rot="R90"/>
 <instance part="GND3" gate="1" x="132.08" y="180.34" rot="R270"/>
 <instance part="GND4" gate="1" x="177.8" y="180.34" rot="R90"/>
@@
 <segment>
 <pinref part="COUNTER" gate="G$1" pin="GND"/>
-<wire x1="81.28" y1="190.5" x2="83.82" y2="190.5" width="0.1524" layer="91"/>
+<wire x1="81.28" y1="187.96" x2="83.82" y2="187.96" width="0.1524" layer="91"/>
 <pinref part="COUNTER" gate="G$1" pin="MR"/>
-<wire x1="81.28" y1="185.42" x2="83.82" y2="185.42" width="0.1524" layer="91"/>
-<wire x1="83.82" y1="190.5" x2="83.82" y2="185.42" width="0.1524" layer="91"/>
-<wire x1="83.82" y1="185.42" x2="86.36" y2="185.42" width="0.1524" layer="91"/>
+<wire x1="81.28" y1="182.88" x2="83.82" y2="182.88" width="0.1524" layer="91"/>
+<wire x1="83.82" y1="187.96" x2="83.82" y2="182.88" width="0.1524" layer="91"/>
+<wire x1="83.82" y1="182.88" x2="86.36" y2="182.88" width="0.1524" layer="91"/>
 <pinref part="GND2" gate="1" pin="GND"/>
 </segment>
@@
 <segment>
 <pinref part="COUNTER" gate="G$1" pin="Q14"/>
-<wire x1="55.88" y1="160.02" x2="53.34" y2="160.02" width="0.1524" layer="91"/>
+<wire x1="55.88" y1="157.48" x2="53.34" y2="157.48" width="0.1524" layer="91"/>
 </segment>
 <segment>
@@
 <segment>
 <pinref part="COUNTER" gate="G$1" pin="VCC"/>
-<wire x1="81.28" y1="195.58" x2="83.82" y2="195.58" width="0.1524" layer="91"/>
-<label x="83.82" y="195.58" size="1.778" layer="95"/>
+<wire x1="81.28" y1="193.04" x2="83.82" y2="193.04" width="0.1524" layer="91"/>
+<label x="83.82" y="193.04" size="1.778" layer="95"/>
 </segment>
 <segment>
@@
 <segment>
 <pinref part="COUNTER" gate="G$1" pin="RTC"/>
-<wire x1="81.28" y1="175.26" x2="83.82" y2="175.26" width="0.1524" layer="91"/>
-<label x="81.28" y="175.26" size="1.778" layer="95"/>
-</segment>
-<segment>
+<wire x1="81.28" y1="172.72" x2="83.82" y2="172.72" width="0.1524" layer="91"/>
+<label x="81.28" y="172.72" size="1.778" layer="95"/>
+</segment>
+<segment>
