File: schematics/chainclock.brd (EAGLE design)
At the start: 55 x 46.5 mm, 21 parts

Commit message: Start on software and v2.0
Parts:
- removed C3, C4: 100uf, SparkFun-Capacitors:CAP-PTH-SMALL-KIT
- added C1, C2: (no value), SparkFun-Capacitors:CPOL-RADIAL-100UF-25V
- moved SG3040JC 14.4 mm to (34.6, 27.6), turned to 180 degrees
Connections:
- removed net N$1: PTN04050.1, R4.P$1
- net GND: now also C1.2, C2.2, PTN04050.1, R4.P$1; no longer C3.2, C4.2
- net VBATT: now also C1.1; no longer C3.1
- net VIN: now also C2.1; no longer C4.1
Routing:
- net N$1: track 15.0 -> 0.00 mm
- net RTC: track 17.8 -> 11.2 mm
- net 3V3: track 76.3 -> 80.2 mm
- net VBATT: track 52.1 -> 54.6 mm
- net VIN: track 57.9 -> 60.2 mm
Changed lines of the file:
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@@
 <setting verticaltext="up"/>
 </settings>
-<grid distance="0.0125" unitdist="inch" unit="mm" style="lines" multiple="1" display="yes" altdistance="0.025" altunitdist="inch" altunit="inch"/>
+<grid distance="0.025" unitdist="inch" unit="inch" style="lines" multiple="1" display="yes" altdistance="0.025" altunitdist="inch" altunit="inch"/>
 <layers>
 <layer number="1" name="Top" color="4" fill="1" visible="yes" active="yes"/>
@@
 <element name="C5" library="SparkFun-Capacitors" package="CAP-PTH-SMALL-KIT" value=".01uf" x="15.24" y="26.67"/>
 <element name="C6" library="SparkFun-Capacitors" package="CAP-PTH-SMALL-KIT" value=".01uf" x="15.24" y="29.21"/>
-<element name="SG3040JC" library="desjardins" package="SG3030JC" value="SG30XXJC" x="24.765" y="17.145"/>
+<element name="SG3040JC" library="desjardins" package="SG3030JC" value="SG30XXJC" x="34.6075" y="27.6225" rot="R180"/>
 <element name="R1" library="SparkFun-Resistors" package="AXIAL-0.3EZ" value="10k" x="15.24" y="38.1" rot="R180"/>
 <element name="R2" library="SparkFun-Resistors" package="AXIAL-0.3EZ" value="10k" x="15.24" y="34.29" rot="R180"/>
@@
 <element name="COUNTER4060_2" library="desjardins" package="SO016" value="4060SOIC16" x="15.875" y="8.89" rot="R90"/>
 <element name="JP3" library="SparkFun-Connectors" package="1X09" value="M09" x="26.67" y="44.45"/>
-<element name="C3" library="SparkFun-Capacitors" package="CAP-PTH-SMALL-KIT" value="100uf" x="43.18" y="14.605" rot="R180">
-<attribute name="PROD_ID" value="CAP-08370" x="43.18" y="14.605" size="1.778" layer="27" rot="R180" display="off"/>
-</element>
-<element name="C4" library="SparkFun-Capacitors" package="CAP-PTH-SMALL-KIT" value="100uf" x="27.305" y="14.605" rot="R180">
-<attribute name="PROD_ID" value="CAP-08370" x="27.305" y="14.605" size="1.778" layer="27" rot="R180" display="off"/>
-</element>
 <element name="JP2" library="SparkFun-Connectors" package="1X09" value="M09" x="4.1275" y="38.1" rot="R270"/>
+<element name="C1" library="SparkFun-Capacitors" package="CPOL-RADIAL-100UF-25V" value="" x="43.815" y="17.145"/>
+<element name="C2" library="SparkFun-Capacitors" package="CPOL-RADIAL-100UF-25V" value="" x="27.305" y="17.145"/>
 </elements>
 <signals>
@@
 <contactref element="JP3" pad="4"/>
 <contactref element="JP3" pad="5"/>
-<contactref element="C3" pad="2"/>
-<contactref element="C4" pad="2"/>
 <contactref element="U$4" pad="P6"/>
 <contactref element="U$4" pad="P31"/>
 <contactref element="JP2" pad="8"/>
+<contactref element="PTN04050" pad="1"/>
+<contactref element="R4" pad="P$1"/>
+<contactref element="C1" pad="2"/>
+<contactref element="C2" pad="2"/>
 </signal>
 <signal name="3V30">
@@
 <wire x1="15.875" y1="6.35" x2="13.97" y2="4.445" width="0.3048" layer="1"/>
 <wire x1="13.97" y1="4.445" x2="13.075" y2="4.445" width="0.3048" layer="1"/>
-<wire x1="27.475" y1="22.745" x2="27.475" y2="18.145" width="0.3048" layer="1"/>
 <wire x1="12.065" y1="4.445" x2="8.89" y2="7.62" width="0.3048" layer="1"/>
 <wire x1="8.89" y1="7.62" x2="8.89" y2="38.735" width="0.3048" layer="1"/>
 <wire x1="8.89" y1="38.735" x2="6.985" y2="40.64" width="0.3048" layer="1"/>
-<wire x1="27.475" y1="22.745" x2="26.785" y2="22.745" width="0.3048" layer="1"/>
-<wire x1="26.785" y1="22.745" x2="25.4" y2="24.13" width="0.3048" layer="1"/>
-<wire x1="25.4" y1="24.13" x2="18.675" y2="24.13" width="0.3048" layer="1"/>
+<wire x1="31.75" y1="22.17" x2="31.75" y2="24.13" width="0.4064" layer="1"/>
+<wire x1="31.75" y1="24.13" x2="31.75" y2="26.475" width="0.4064" layer="1"/>
+<wire x1="31.75" y1="26.475" x2="31.8975" y2="26.6225" width="0.4064" layer="1"/>
+<wire x1="31.75" y1="22.17" x2="31.8975" y2="22.0225" width="0.4064" layer="1"/>
+<wire x1="18.675" y1="24.13" x2="31.75" y2="24.13" width="0.3048" layer="1"/>
 </signal>
 <signal name="RENB">
@@
 <contactref element="SG3040JC" pad="3"/>
 <contactref element="COUNTER4060_1" pad="10"/>
-<wire x1="18.675" y1="16.51" x2="28.575" y2="16.51" width="0.3048" layer="1"/>
-<wire x1="28.575" y1="16.51" x2="30.48" y2="18.415" width="0.3048" layer="1"/>
-<wire x1="30.48" y1="18.415" x2="30.48" y2="20.67" width="0.3048" layer="1"/>
-<wire x1="30.48" y1="20.67" x2="32.555" y2="22.745" width="0.3048" layer="1"/>
+<wire x1="18.675" y1="16.51" x2="19.685" y2="16.51" width="0.3048" layer="1"/>
+<wire x1="19.685" y1="16.51" x2="20.32" y2="17.145" width="0.3048" layer="1"/>
+<wire x1="20.32" y1="17.145" x2="20.32" y2="18.415" width="0.3048" layer="1"/>
+<wire x1="20.32" y1="18.415" x2="20.955" y2="19.05" width="0.3048" layer="1"/>
+<wire x1="20.955" y1="19.05" x2="23.845" y2="19.05" width="0.3048" layer="1"/>
+<wire x1="23.845" y1="19.05" x2="26.8175" y2="22.0225" width="0.3048" layer="1"/>
 </signal>
 <signal name="VIN">
@@
 <wire x1="12.7" y1="2.54" x2="7.62" y2="7.62" width="0.3048" layer="16"/>
 <wire x1="7.62" y1="7.62" x2="6.985" y2="7.62" width="0.3048" layer="16"/>
-<contactref element="C4" pad="1"/>
 <wire x1="25.781" y1="2.286" x2="28.575" y2="5.08" width="0.3048" layer="16"/>
-<wire x1="28.575" y1="5.08" x2="28.575" y2="14.478" width="0.3048" layer="16"/>
-<wire x1="28.575" y1="14.478" x2="28.702" y2="14.605" width="0.3048" layer="16"/>
 <wire x1="44.45" y1="30.099" x2="44.45" y2="29.845" width="0.3048" layer="16"/>
-<wire x1="44.45" y1="29.845" x2="31.75" y2="17.145" width="0.3048" layer="16"/>
-<wire x1="31.75" y1="17.145" x2="31.242" y2="17.145" width="0.3048" layer="16"/>
-<wire x1="31.242" y1="17.145" x2="28.702" y2="14.605" width="0.3048" layer="16"/>
+<contactref element="C2" pad="1"/>
+<wire x1="44.45" y1="29.845" x2="38.1" y2="23.495" width="0.4064" layer="16"/>
+<wire x1="38.1" y1="23.495" x2="38.1" y2="22.225" width="0.4064" layer="16"/>
+<wire x1="38.1" y1="22.225" x2="33.02" y2="17.145" width="0.4064" layer="16"/>
+<wire x1="33.02" y1="17.145" x2="28.575" y2="17.145" width="0.4064" layer="16"/>
+<wire x1="28.575" y1="5.08" x2="28.575" y2="17.145" width="0.4064" layer="16"/>
 </signal>
 <signal name="REF">
@@
 <wire x1="31.115" y1="14.605" x2="31.4325" y2="14.9225" width="0.3048" layer="1"/>
 </signal>
-<signal name="N$1">
-<contactref element="PTN04050" pad="1"/>
-<contactref element="R4" pad="P$1"/>
-<wire x1="39.0525" y1="14.9225" x2="39.0525" y2="8.0645" width="0.3048" layer="16"/>
-<wire x1="39.0525" y1="8.0645" x2="44.831" y2="2.286" width="0.3048" layer="16"/>
-</signal>
 <signal name="VBATT">
 <contactref element="PTN04050" pad="2"/>
@@
 <wire x1="11.43" y1="3.175" x2="19.685" y2="3.175" width="0.3048" layer="1"/>
 <wire x1="19.685" y1="3.175" x2="20.32" y2="3.81" width="0.3048" layer="1"/>
-<contactref element="C3" pad="1"/>
 <wire x1="20.32" y1="3.81" x2="40.005" y2="3.81" width="0.3048" layer="1"/>
+<contactref element="C1" pad="1"/>
 <wire x1="40.005" y1="3.81" x2="44.831" y2="8.636" width="0.3048" layer="1"/>
-<wire x1="44.577" y1="14.605" x2="44.577" y2="8.89" width="0.3048" layer="1"/>
-<wire x1="44.577" y1="8.89" x2="44.831" y2="8.636" width="0.3048" layer="1"/>
+<wire x1="45.085" y1="17.145" x2="45.085" y2="8.89" width="0.3048" layer="1"/>
+<wire x1="45.085" y1="8.89" x2="44.831" y2="8.636" width="0.3048" layer="1"/>
 </signal>
 <signal name="Q13">
