File: schematics/chainclock.sch (EAGLE design)
At the start: 18 parts

Commit message: Update layout of chainclock
Connections:
- net 3A: now also U$4.D12; no longer U$4.D11
- net 4A: now also U$4.D11; no longer U$4.D12
Changed lines of the file:
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@@
 </segment>
 <segment>
-<pinref part="U$4" gate="G$1" pin="D12"/>
-<wire x1="134.62" y1="91.44" x2="132.08" y2="91.44" width="0.1524" layer="91"/>
-<label x="132.08" y="93.98" size="1.778" layer="95" rot="R180"/>
+<pinref part="U$4" gate="G$1" pin="D11"/>
+<wire x1="134.62" y1="93.98" x2="132.08" y2="93.98" width="0.1524" layer="91"/>
+<label x="132.08" y="96.52" size="1.778" layer="95" rot="R180"/>
 </segment>
 </net>
@@
 </segment>
 <segment>
-<pinref part="U$4" gate="G$1" pin="D11"/>
-<wire x1="134.62" y1="93.98" x2="132.08" y2="93.98" width="0.1524" layer="91"/>
-<label x="132.08" y="96.52" size="1.778" layer="95" rot="R180"/>
+<pinref part="U$4" gate="G$1" pin="D12"/>
+<wire x1="134.62" y1="91.44" x2="132.08" y2="91.44" width="0.1524" layer="91"/>
+<label x="132.08" y="93.98" size="1.778" layer="95" rot="R180"/>
 </segment>
 </net>

Commit message: First pass
Parts:
- added JP2: M09, SparkFun-Connectors:M09
- renumbered U$1 to PTN04050
Connections:
- new net A0: JP2.2, U$4.A0
- new net A1: JP2.3, U$4.A1
- new net A2: JP2.4, U$4.A2
- new net A3: JP2.5, U$4.A3
- new net A4: JP2.6, U$4.A4
- new net A5: JP2.7, U$4.A5
- new net D13: JP2.1, U$4.D13
- net 5VREG: now also JP2.9
- net GND: now also JP2.8
Changed lines of the file:
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@@
 <?xml version="1.0" encoding="utf-8"?>
 <!DOCTYPE eagle SYSTEM "eagle.dtd">
-<eagle version="6.5.0">
+<eagle version="7.4.0">
 <drawing>
 <settings>
@@
 <part name="R8" library="SparkFun-Resistors" deviceset="RESISTOR" device="EZ" value="10k"/>
 <part name="U$4" library="ChrisD" deviceset="ARDUINO_PRO_MICRO" device=""/>
-<part name="U$1" library="desjardins" deviceset="PTN0405C" device=""/>
+<part name="PTN04050" library="desjardins" deviceset="PTN0405C" device=""/>
 <part name="R4" library="SparkFun-Resistors" deviceset="RESISTOR" device="EZ" value="12k"/>
 <part name="GND6" library="SparkFun-Aesthetics" deviceset="GND" device=""/>
@@
 <part name="GND7" library="SparkFun-Aesthetics" deviceset="GND" device=""/>
 <part name="GND12" library="SparkFun-Aesthetics" deviceset="GND" device=""/>
+<part name="JP2" library="SparkFun-Connectors" deviceset="M09" device=""/>
 </parts>
 <sheets>
@@
 <instance part="R8" gate="G$1" x="58.42" y="96.52"/>
 <instance part="U$4" gate="G$1" x="147.32" y="116.84"/>
-<instance part="U$1" gate="G$1" x="213.36" y="134.62"/>
+<instance part="PTN04050" gate="G$1" x="213.36" y="134.62"/>
 <instance part="R4" gate="G$1" x="187.96" y="139.7" rot="R180"/>
 <instance part="GND6" gate="1" x="241.3" y="111.76"/>
@@
 <instance part="GND7" gate="1" x="119.38" y="119.38" rot="MR90"/>
 <instance part="GND12" gate="1" x="167.64" y="124.46" rot="MR270"/>
+<instance part="JP2" gate="G$1" x="172.72" y="66.04"/>
 </instances>
 <busses>
@@
 <pinref part="HBRIDGE" gate="G$1" pin="GND@1"/>
 <wire x1="137.16" y1="180.34" x2="139.7" y2="180.34" width="0.1524" layer="91"/>
-<wire x1="139.7" y1="180.34" x2="134.62" y2="180.34" width="0.1524" layer="91"/>
+<wire x1="139.7" y1="180.34" x2="137.16" y2="180.34" width="0.1524" layer="91"/>
 <pinref part="GND3" gate="1" pin="GND"/>
+<junction x="137.16" y="180.34"/>
+<wire x1="137.16" y1="180.34" x2="134.62" y2="180.34" width="0.1524" layer="91"/>
+<junction x="139.7" y="180.34"/>
 </segment>
 <segment>
@@
 <pinref part="HBRIDGE" gate="G$1" pin="GND@2"/>
 <wire x1="172.72" y1="180.34" x2="170.18" y2="180.34" width="0.1524" layer="91"/>
-<wire x1="170.18" y1="180.34" x2="175.26" y2="180.34" width="0.1524" layer="91"/>
+<wire x1="170.18" y1="180.34" x2="172.72" y2="180.34" width="0.1524" layer="91"/>
 <pinref part="GND4" gate="1" pin="GND"/>
+<junction x="172.72" y="180.34"/>
+<wire x1="172.72" y1="180.34" x2="175.26" y2="180.34" width="0.1524" layer="91"/>
+<junction x="170.18" y="180.34"/>
 </segment>
 <segment>
@@
 <wire x1="48.26" y1="180.34" x2="50.8" y2="180.34" width="0.1524" layer="91"/>
 <pinref part="GND9" gate="1" pin="GND"/>
+<junction x="48.26" y="180.34"/>
 </segment>
 <segment>
@@
 <wire x1="48.26" y1="121.92" x2="50.8" y2="121.92" width="0.1524" layer="91"/>
 <pinref part="GND2" gate="1" pin="GND"/>
+<junction x="48.26" y="121.92"/>
 </segment>
 <segment>
@@
 <pinref part="GND12" gate="1" pin="GND"/>
 </segment>
+<segment>
+<pinref part="JP2" gate="G$1" pin="8"/>
+<wire x1="182.88" y1="73.66" x2="185.42" y2="73.66" width="0.1524" layer="91"/>
+<label x="182.88" y="73.66" size="1.778" layer="95"/>
+</segment>
 </net>
 <net name="CLOCKIN" class="0">
@@
 </segment>
 <segment>
-<pinref part="U$1" gate="G$1" pin="VOUT"/>
+<pinref part="PTN04050" gate="G$1" pin="VOUT"/>
 <wire x1="231.14" y1="139.7" x2="241.3" y2="139.7" width="0.1524" layer="91"/>
 <wire x1="241.3" y1="139.7" x2="243.84" y2="139.7" width="0.1524" layer="91"/>
@@
 <label x="68.58" y="116.84" size="1.778" layer="95"/>
 </segment>
+<segment>
+<pinref part="JP2" gate="G$1" pin="9"/>
+<wire x1="182.88" y1="76.2" x2="185.42" y2="76.2" width="0.1524" layer="91"/>
+<label x="182.88" y="76.2" size="1.778" layer="95"/>
+</segment>
 </net>
 <net name="N$1" class="0">
 <segment>
-<pinref part="U$1" gate="G$1" pin="GND"/>
+<pinref part="PTN04050" gate="G$1" pin="GND"/>
 <wire x1="195.58" y1="139.7" x2="193.04" y2="139.7" width="0.1524" layer="91"/>
 <pinref part="R4" gate="G$1" pin="1"/>
@@
 </segment>
 <segment>
-<pinref part="U$1" gate="G$1" pin="VOADJ"/>
+<pinref part="PTN04050" gate="G$1" pin="VOADJ"/>
 <wire x1="231.14" y1="129.54" x2="233.68" y2="129.54" width="0.1524" layer="91"/>
 <label x="231.14" y="129.54" size="1.778" layer="95"/>
@@
 <net name="VBATT" class="0">
 <segment>
-<pinref part="U$1" gate="G$1" pin="VIN"/>
+<pinref part="PTN04050" gate="G$1" pin="VIN"/>
 <wire x1="195.58" y1="132.08" x2="193.04" y2="132.08" width="0.1524" layer="91"/>
 <wire x1="193.04" y1="132.08" x2="190.5" y2="132.08" width="0.1524" layer="91"/>
@@
 </segment>
 </net>
+<net name="D13" class="0">
+<segment>
+<pinref part="U$4" gate="G$1" pin="D13"/>
+<wire x1="162.56" y1="91.44" x2="165.1" y2="91.44" width="0.1524" layer="91"/>
+<label x="165.1" y="91.44" size="1.778" layer="95"/>
+</segment>
+<segment>
+<pinref part="JP2" gate="G$1" pin="1"/>
+<wire x1="182.88" y1="55.88" x2="185.42" y2="55.88" width="0.1524" layer="91"/>
+<label x="182.88" y="55.88" size="1.778" layer="95"/>
+</segment>
+</net>
+<net name="A0" class="0">
+<segment>
+<pinref part="U$4" gate="G$1" pin="A0"/>
+<wire x1="162.56" y1="99.06" x2="165.1" y2="99.06" width="0.1524" layer="91"/>
+<label x="165.1" y="99.06" size="1.778" layer="95"/>
+</segment>
+<segment>
+<pinref part="JP2" gate="G$1" pin="2"/>
+<wire x1="182.88" y1="58.42" x2="185.42" y2="58.42" width="0.1524" layer="91"/>
+<label x="182.88" y="58.42" size="1.778" layer="95"/>
+</segment>
+</net>
+<net name="A1" class="0">
+<segment>
+<pinref part="U$4" gate="G$1" pin="A1"/>
+<wire x1="162.56" y1="101.6" x2="165.1" y2="101.6" width="0.1524" layer="91"/>
+<label x="165.1" y="101.6" size="1.778" layer="95"/>
+</segment>
+<segment>
+<pinref part="JP2" gate="G$1" pin="3"/>
+<wire x1="182.88" y1="60.96" x2="185.42" y2="60.96" width="0.1524" layer="91"/>
+<label x="182.88" y="60.96" size="1.778" layer="95"/>
+</segment>
+</net>
+<net name="A2" class="0">
+<segment>
+<pinref part="U$4" gate="G$1" pin="A2"/>
+<wire x1="162.56" y1="104.14" x2="165.1" y2="104.14" width="0.1524" layer="91"/>
+<label x="165.1" y="104.14" size="1.778" layer="95"/>
+</segment>
+<segment>
+<pinref part="JP2" gate="G$1" pin="4"/>
+<wire x1="182.88" y1="63.5" x2="185.42" y2="63.5" width="0.1524" layer="91"/>
+<label x="182.88" y="63.5" size="1.778" layer="95"/>
+</segment>
+</net>
+<net name="A3" class="0">
+<segment>
+<pinref part="U$4" gate="G$1" pin="A3"/>
+<wire x1="162.56" y1="106.68" x2="165.1" y2="106.68" width="0.1524" layer="91"/>
+<label x="165.1" y="106.68" size="1.778" layer="95"/>
+</segment>
+<segment>
+<pinref part="JP2" gate="G$1" pin="5"/>
+<wire x1="182.88" y1="66.04" x2="185.42" y2="66.04" width="0.1524" layer="91"/>
+<label x="182.88" y="66.04" size="1.778" layer="95"/>
+</segment>
+</net>
+<net name="A4" class="0">
+<segment>
+<pinref part="U$4" gate="G$1" pin="A4"/>
+<wire x1="162.56" y1="109.22" x2="165.1" y2="109.22" width="0.1524" layer="91"/>
+<label x="165.1" y="109.22" size="1.778" layer="95"/>
+</segment>
+<segment>
+<pinref part="JP2" gate="G$1" pin="6"/>
+<wire x1="182.88" y1="68.58" x2="185.42" y2="68.58" width="0.1524" layer="91"/>
+<label x="182.88" y="68.58" size="1.778" layer="95"/>
+</segment>
+</net>
+<net name="A5" class="0">
+<segment>
+<pinref part="U$4" gate="G$1" pin="A5"/>
+<wire x1="162.56" y1="111.76" x2="165.1" y2="111.76" width="0.1524" layer="91"/>
+<label x="165.1" y="111.76" size="1.778" layer="95"/>
+</segment>
+<segment>
+<pinref part="JP2" gate="G$1" pin="7"/>
+<wire x1="182.88" y1="71.12" x2="185.42" y2="71.12" width="0.1524" layer="91"/>
+<label x="182.88" y="71.12" size="1.778" layer="95"/>
+</segment>
+</net>
 </nets>
 </sheet>
 </sheets>
+<errors>
+</errors>
 </schematic>
 </drawing>

Commit message: Start on software and v2.0
Parts:
- removed C3, C4: 100uf, SparkFun-Capacitors:0.1UF-50V-20%(PTH)KIT-EZ
- added C1, C2: (no value), SparkFun-Capacitors:CAP_POLPTH1
Connections:
- removed net N$1: PTN04050.GND, R4.1
- net GND: now also C1.-, C2.-, PTN04050.GND, R4.1; no longer C3.2, C4.2
- net VBATT: now also C1.+; no longer C3.1
- net VIN: now also C2.+; no longer C4.1
Other:
- moved on the sheet: R4
Changed lines of the file:
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@@
 <part name="JP3" library="SparkFun-Connectors" deviceset="M09" device=""/>
 <part name="GND14" library="SparkFun-Aesthetics" deviceset="GND" device=""/>
-<part name="C3" library="SparkFun-Capacitors" deviceset="0.1UF-50V-20%(PTH)" device="KIT-EZ" value="100uf"/>
-<part name="C4" library="SparkFun-Capacitors" deviceset="0.1UF-50V-20%(PTH)" device="KIT-EZ" value="100uf"/>
 <part name="GND7" library="SparkFun-Aesthetics" deviceset="GND" device=""/>
 <part name="GND12" library="SparkFun-Aesthetics" deviceset="GND" device=""/>
 <part name="JP2" library="SparkFun-Connectors" deviceset="M09" device=""/>
+<part name="GND13" library="SparkFun-Aesthetics" deviceset="GND" device=""/>
+<part name="C1" library="SparkFun-Capacitors" deviceset="CAP_POL" device="PTH1"/>
+<part name="C2" library="SparkFun-Capacitors" deviceset="CAP_POL" device="PTH1"/>
 </parts>
 <sheets>
@@
 <instance part="U$4" gate="G$1" x="147.32" y="116.84"/>
 <instance part="PTN04050" gate="G$1" x="213.36" y="134.62"/>
-<instance part="R4" gate="G$1" x="187.96" y="139.7" rot="R180"/>
+<instance part="R4" gate="G$1" x="185.42" y="139.7" rot="R180"/>
 <instance part="GND6" gate="1" x="241.3" y="111.76"/>
 <instance part="GND8" gate="1" x="193.04" y="111.76"/>
@@
 <instance part="JP3" gate="G$1" x="109.22" y="68.58"/>
 <instance part="GND14" gate="1" x="142.24" y="68.58" rot="MR270"/>
-<instance part="C3" gate="G$1" x="193.04" y="119.38"/>
-<instance part="C4" gate="G$1" x="241.3" y="119.38"/>
 <instance part="GND7" gate="1" x="119.38" y="119.38" rot="MR90"/>
 <instance part="GND12" gate="1" x="167.64" y="124.46" rot="MR270"/>
 <instance part="JP2" gate="G$1" x="172.72" y="66.04"/>
+<instance part="GND13" gate="1" x="193.04" y="144.78" rot="R180"/>
+<instance part="C1" gate="G$1" x="193.04" y="121.92"/>
+<instance part="C2" gate="G$1" x="241.3" y="121.92"/>
 </instances>
 <busses>
@@
 <wire x1="241.3" y1="116.84" x2="241.3" y2="114.3" width="0.1524" layer="91"/>
 <pinref part="GND6" gate="1" pin="GND"/>
-<pinref part="C4" gate="G$1" pin="2"/>
+<pinref part="C2" gate="G$1" pin="-"/>
 </segment>
 <segment>
 <wire x1="193.04" y1="116.84" x2="193.04" y2="114.3" width="0.1524" layer="91"/>
 <pinref part="GND8" gate="1" pin="GND"/>
-<pinref part="C3" gate="G$1" pin="2"/>
+<pinref part="C1" gate="G$1" pin="-"/>
 </segment>
 <segment>
@@
 <label x="182.88" y="73.66" size="1.778" layer="95"/>
 </segment>
+<segment>
+<pinref part="PTN04050" gate="G$1" pin="GND"/>
+<wire x1="195.58" y1="139.7" x2="193.04" y2="139.7" width="0.1524" layer="91"/>
+<pinref part="R4" gate="G$1" pin="1"/>
+<wire x1="193.04" y1="139.7" x2="190.5" y2="139.7" width="0.1524" layer="91"/>
+<wire x1="193.04" y1="139.7" x2="193.04" y2="142.24" width="0.1524" layer="91"/>
+<pinref part="GND13" gate="1" pin="GND"/>
+<junction x="193.04" y="139.7"/>
+</segment>
 </net>
 <net name="CLOCKIN" class="0">
@@
 <junction x="241.3" y="139.7"/>
 <label x="243.84" y="139.7" size="1.778" layer="95"/>
-<pinref part="C4" gate="G$1" pin="1"/>
+<pinref part="C2" gate="G$1" pin="+"/>
 </segment>
 </net>
@@
 </segment>
 </net>
-<net name="N$1" class="0">
-<segment>
-<pinref part="PTN04050" gate="G$1" pin="GND"/>
-<wire x1="195.58" y1="139.7" x2="193.04" y2="139.7" width="0.1524" layer="91"/>
-<pinref part="R4" gate="G$1" pin="1"/>
-</segment>
-</net>
 <net name="VOADJ" class="0">
 <segment>
 <pinref part="R4" gate="G$1" pin="2"/>
-<wire x1="182.88" y1="139.7" x2="180.34" y2="139.7" width="0.1524" layer="91"/>
+<wire x1="180.34" y1="139.7" x2="177.8" y2="139.7" width="0.1524" layer="91"/>
 <label x="175.26" y="139.7" size="1.778" layer="95"/>
 </segment>
@@
 <junction x="193.04" y="132.08"/>
 <label x="182.88" y="132.08" size="1.778" layer="95"/>
-<pinref part="C3" gate="G$1" pin="1"/>
-</segment>
-<segment>
+<pinref part="C1" gate="G$1" pin="+"/>
+</segment>
+<segment>
